File: Hardware/Arduino controlled radio.kicad_pcb (KiCad board)
At the start: 2 copper layers, 92.1 x 92.1 mm, 74 parts, among them J1 Jack-DC, J2 Conn_02x15_Odd_Even, J3 Conn_01x02, J4 HC-06 Connector, J5 Conn_Coaxial, J6 Conn_01x02, J7 SJ1-3525NG, J8 Speaker, Q1 2N7002, Q2 2N7002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

Commit message: Rev 3 Boards
Parts:
- removed C17: .1uF, Capacitor_SMD:C_0805_2012Metric_Pad1.18x1.45mm_HandSolder
- removed C18: 100uF 16V, Capacitor_SMD:CP_Elec_6.3x7.7
- removed C19: .22uF, Capacitor_SMD:C_0805_2012Metric_Pad1.15x1.40mm_HandSolder
- removed C20: 2200uF 16V, Capacitor_THT:CP_Radial_D12.5mm_P5.00mm
- removed Q4, Q5: BC847, Package_TO_SOT_SMD:SOT-23
- removed R19: 470K, Resistor_SMD:R_0805_2012Metric_Pad1.15x1.40mm_HandSolder
- removed R20, R22, R23, R24: 22K, Resistor_SMD:R_0805_2012Metric_Pad1.15x1.40mm_HandSolder
- removed R21: 2.2K, Resistor_SMD:R_0805_2012Metric_Pad1.15x1.40mm_HandSolder
- removed R25: 1ohm 1.2W, Resistor_THT:R_Axial_DIN0411_L9.9mm_D3.6mm_P15.24mm_Horizontal
- removed TP4, TP5, TP8: TestPoint, TestPoint:TestPoint_Keystone_5000-5004_Miniature
- added REF**: MountingHole_4.3mm_M4, MountingHole:MountingHole_4.3mm_M4, F.Cu at (90.1, 44.2)
- added REF**: MountingHole_4.3mm_M4, MountingHole:MountingHole_4.3mm_M4, F.Cu at (170.1, 44.2)
- added REF**: MountingHole_4.3mm_M4, MountingHole:MountingHole_4.3mm_M4, F.Cu at (170.1, 124.2)
- added REF**: MountingHole_4.3mm_M4, MountingHole:MountingHole_4.3mm_M4, F.Cu at (89.8, 124.2)
- added U4: TPA3118AmplifierBoard, Arduino controlled radio:TPA3118_Board, F.Cu at (120.4, 104.6)
- C10, C11: value 10uF 16V -> 1uF; footprint Capacitor_SMD:CP_Elec_4x5.3 -> Capacitor_SMD:C_0805_2012Metric_Pad1.15x1.40mm_HandSolder
- C12: value 10uF 16V -> .1uF; footprint Capacitor_SMD:CP_Elec_4x5.3 -> Capacitor_SMD:C_0805_2012Metric_Pad1.15x1.40mm_HandSolder
- C13, C14: value 10uF 16V -> 10uF; footprint Capacitor_SMD:CP_Elec_4x5.3 -> Capacitor_SMD:C_0805_2012Metric_Pad1.15x1.40mm_HandSolder
- C15: value 10uF 16V -> 100uF; footprint Capacitor_SMD:CP_Elec_4x5.3 -> Capacitor_SMD:C_Elec_6.3x5.4
- C16: value 1uF -> .1 uF; footprint Capacitor_SMD:C_0805_2012Metric_Pad1.18x1.45mm_HandSolder -> Capacitor_SMD:C_0805_2012Metric_Pad1.15x1.40mm_HandSolder
- J2: moved to F.Cu
- R11, R13: value 20K -> 22K
- R12, R14: value 18K -> 22K
- R15, R16: value 390 -> 22K
- R17, R18: value 470 -> 1K
- R2: footprint Resistor_THT:R_Axial_DIN0204_L3.6mm_D1.6mm_P7.62mm_Horizontal -> Resistor_SMD:R_0805_2012Metric_Pad1.15x1.40mm_HandSolder
- U3: value LM1875 -> LM358; footprint Package_TO_SOT_THT:TO-220-5_P3.4x3.7mm_StaggerOdd_Lead3.8mm_Vertical -> Arduino controlled radio:TL082CDR
- Y1: footprint Arduino controlled radio:XTAL_ECS-.327-12.5-12-C-TR -> Crystal:Crystal_AT310_D3.0mm_L10.0mm_Vertical
- moved C14 124.8 mm to (128.8, 78.7)
- moved C15 118.3 mm to (125.7, 86.9), turned to 0 degrees
- moved C16 115.7 mm to (111.3, 54.9)
- moved U3 37.5 mm to (127.9, 68.7), turned to 270 degrees
- moved R10 33.7 mm to (164.8, 80.9), turned to 90 degrees
- moved C13 23.4 mm to (129.3, 58.2), turned to 0 degrees
- moved D1 20.3 mm to (153.1, 57.0), turned to 90 degrees
- moved R12 14.2 mm to (134.9, 69.8), turned to 180 degrees
- moved C12 13.9 mm to (124.2, 58.2), turned to 0 degrees
- moved R11 12.0 mm to (134.9, 65.8), turned to 180 degrees
- moved L2 11.3 mm to (141.5, 50.9)
- moved R16 10.8 mm to (128.8, 75.2), turned to 0 degrees
- moved C11 10.8 mm to (139.2, 69.8), turned to 0 degrees
- moved R15 10.4 mm to (129.3, 62.2), turned to 0 degrees
- moved C10 10.0 mm to (139.2, 65.8), turned to 0 degrees
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Connections:
- C10 pad 1: RChan -> Net-(C10-Pad1)
- C10 pad 2: Net-(C10-Pad2) -> RChan
- C11 pad 1: LChan -> Net-(C11-Pad1)
- C11 pad 2: Net-(C11-Pad2) -> LChan
- C12 pad 1: Net-(C12-Pad1) -> GNDREF
- C14 pad 2: GNDREF -> Net-(C14-Pad2)
- C15 pad 1: Net-(C15-Pad1) -> +12V
- C16 pad 1: Net-(C16-Pad1) -> GNDREF
- C16 pad 2: Net-(C16-Pad2) -> +12V
- J7 pad 2: Net-(C12-Pad2) -> Net-(C13-Pad1)
- J7 pad 3: Net-(C13-Pad2) -> Net-(C14-Pad1)
- J8 pad 2: GNDREF -> Net-(J8-Pad2)
- R11 pad 1: Net-(C10-Pad2) -> Net-(C10-Pad1)
- R11 pad 2: +5V -> Net-(R11-Pad2)
- R12 pad 1: Net-(C12-Pad1) -> Net-(C11-Pad1)
- R12 pad 2: Net-(C10-Pad2) -> Net-(R12-Pad2)
- R13 pad 1: Net-(C11-Pad2) -> Net-(C12-Pad2)
- R13 pad 2: +5V -> +12V
- R14 pad 1: Net-(C13-Pad1) -> GNDREF
- R14 pad 2: Net-(C11-Pad2) -> Net-(C12-Pad2)
- R15 pad 1: GNDREF -> Net-(R11-Pad2)
- R15 pad 2: Net-(C12-Pad1) -> Net-(C13-Pad2)
- R16 pad 1: GNDREF -> Net-(R12-Pad2)
- R16 pad 2: Net-(C13-Pad1) -> Net-(C14-Pad2)
- R17 pad 1: Net-(C16-Pad2) -> Net-(J7-Pad5)
- R17 pad 2: Net-(J7-Pad4) -> Net-(R17-Pad2)
- R18 pad 1: Net-(C16-Pad2) -> Net-(J7-Pad4)
- R18 pad 2: Net-(J7-Pad5) -> Net-(R17-Pad2)
- U3 pad 1: Net-(C16-Pad1) -> Net-(C13-Pad2)
- U3 pad 2: Net-(R21-Pad1) -> Net-(R11-Pad2)
- U3 pad 3: GNDREF -> Net-(C12-Pad2)
- U3 pad 4: Net-(C20-Pad1) -> GNDREF
- U3 pad 5: +12V -> Net-(C12-Pad2)
Routing:
- net +5V: track 3.06 -> 189.0 mm, vias 0 -> 6
- net +12V: track 0.00 -> 130.6 mm
- net +3V3: track 0.00 -> 68.9 mm, vias 0 -> 3
- net Net-(R17-Pad2): track 0.00 -> 67.9 mm
- net GNDREF: track 8.32 -> 70.9 mm, vias 0 -> 9
- net GNDA: track 0.00 -> 44.5 mm
- net Net-(C14-Pad1): track 0.00 -> 32.2 mm
- net Net-(J1-Pad1): track 0.00 -> 28.7 mm
- net Net-(C13-Pad1): track 0.00 -> 25.1 mm
- net Net-(C12-Pad2): track 0.00 -> 20.2 mm
- net Net-(J8-Pad2): track 0.00 -> 19.5 mm
- net Net-(C8-Pad1): track 0.00 -> 18.0 mm
- net Net-(C7-Pad1): track 1.92 -> 18.0 mm
- net Net-(J8-Pad1): track 0.00 -> 14.3 mm
- net Net-(R12-Pad2): track 0.00 -> 12.3 mm
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- added copper zone on B.Cu, net GNDREF
Other:
- net class Default: trace_width 0.6 -> 0.203; via_dia 0.8 -> 0.56; via_drill 0.4 -> 0.33
- net class Medium Power added: clearance 0.2, trace_width 0.381, via_dia 0.8, via_drill 0.4
- board text added: "1"
