File: Hardware/Arduino controlled radio.sch (KiCad schematic (older format))
At the start: 40 parts, among them J1 Jack-DC, J2 Conn_02x15_Odd_Even, J3 Conn_01x02, J4 HC-06 Connector, J5 Conn_Coaxial, J6 Conn_01x02, Q1 2N7002, Q2 2N7002, Q3 2N7002, U1 NE555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

Commit message: Rev 3 Boards
Parts:
- R2: footprint Resistor_THT:R_Axial_DIN0204_L3.6mm_D1.6mm_P7.62mm_Horizontal -> Resistor_SMD:R_0805_2012Metric_Pad1.15x1.40mm_HandSolder
- Y1: footprint Arduino controlled radio:XTAL_ECS-.327-12.5-12-C-TR -> Crystal:Crystal_AT310_D3.0mm_L10.0mm_Vertical
Changed lines of the file:
@@
 F 0 "Y1" V 7079 4263 50  0000 L CNN
 F 1 "32768KHz" V 7325 3925 50  0000 L CNN
-F 2 "Arduino controlled radio:XTAL_ECS-.327-12.5-12-C-TR" H 7125 4175 50  0001 C CNN
+F 2 "Crystal:Crystal_AT310_D3.0mm_L10.0mm_Vertical" H 7125 4175 50  0001 C CNN
 F 3 "~" H 7125 4175 50  0001 C CNN
 	1    7125 4175
@@
 F 0 "R2" H 4000 6200 50  0000 L CNN
 F 1 "1Meg" H 4125 6200 50  0000 L CNN
-F 2 "Resistor_THT:R_Axial_DIN0204_L3.6mm_D1.6mm_P7.62mm_Horizontal" H 4125 5925 50  0001 C CNN
+F 2 "Resistor_SMD:R_0805_2012Metric_Pad1.15x1.40mm_HandSolder" H 4125 5925 50  0001 C CNN
 F 3 "~" H 4125 5925 50  0001 C CNN
 	1    4125 5925

Commit message: Initial upload of PC Client
Parts:
- removed Q1, Q2, Q3: 2N7002, Package_TO_SOT_SMD:SOT-23, symbol Transistor_FET:2N7002
- added C10, C11: 10uF, Capacitor_SMD:C_0805_2012Metric_Pad1.15x1.40mm_HandSolder, symbol Device:C_Small
- added C12: 100uF, Capacitor_SMD:C_Elec_6.3x5.4, symbol Device:CP1_Small
- added C13: .1 uF, Capacitor_SMD:C_0805_2012Metric_Pad1.15x1.40mm_HandSolder, symbol Device:C_Small
- added C14: .1uF, Capacitor_SMD:C_0805_2012Metric_Pad1.15x1.40mm_HandSolder, symbol Device:C_Small
- added J7: SJ1-3525NG, Arduino controlled radio:CUI_SJ1-3525NG, symbol Arduino~Controlled~Radio:SJ1-3525NG
- added J8: Speaker, Arduino controlled radio:CUI_RCJ-045, symbol Connector:Conn_Coaxial
- added R11: 2.2k, Resistor_SMD:R_0805_2012Metric_Pad1.15x1.40mm_HandSolder, symbol Device:R_Small_US
- added U3: TPA3118AmplifierBoard, Arduino controlled radio:TPA3118_Board, symbol Arduino~Controlled~Radio:TPA3118AmplifierBoard
- A1: value Arduino_BLE_Nano -> Arduino_Nano
- R3, R6: value 10K -> 1K
- R7: value 10K -> 2.2K
Connections:
- wire segments 236 -> 264
Other:
- moved on the sheet: R4, R5
