File: Hardware/Audio Amplifier.sch (KiCad schematic (older format))
At the start: 60 parts, among them J7 SJ1-3525NG, J8 Speaker, Q4 BC847, Q5 BC847, U3 LM1875

Commit message: Initial upload of PC Client
Parts:
- removed C10, C11, C12, C13, C14: 10uF 16V, Capacitor_SMD:CP_Elec_4x5.3, symbol Device:CP1_Small
- removed C17, C?: .1uF, Capacitor_SMD:C_0805_2012Metric_Pad1.18x1.45mm_HandSolder, symbol Device:C_Small
- removed C18, C?: 100uF 16V, Capacitor_SMD:CP_Elec_6.3x7.7, symbol Device:CP1_Small
- removed C19, C?: .22uF, Capacitor_SMD:C_0805_2012Metric_Pad1.15x1.40mm_HandSolder, symbol Device:C_Small
- removed C20, C?: 2200uF 16V, Capacitor_THT:CP_Radial_D12.5mm_P5.00mm, symbol Device:CP1_Small
- removed C? (x2): 10uF, Capacitor_SMD:C_0805_2012Metric_Pad1.18x1.45mm_HandSolder, symbol Device:C_Small
- removed J7: SJ1-3525NG, Arduino controlled radio:CUI_SJ1-3525NG, symbol Arduino~Controlled~Radio:SJ1-3525NG
- removed J8: Speaker, Arduino controlled radio:CUI_RCJ-045, symbol Connector:Conn_Coaxial
- removed Q4, Q5: BC847, Package_TO_SOT_SMD:SOT-23, symbol Transistor_BJT:BC847
- removed R11, R13: 20K, Resistor_SMD:R_0805_2012Metric_Pad1.15x1.40mm_HandSolder, symbol Device:R_Small_US
- removed R12, R14: 18K, Resistor_SMD:R_0805_2012Metric_Pad1.15x1.40mm_HandSolder, symbol Device:R_Small_US
- removed R15, R16: 390, Resistor_SMD:R_0805_2012Metric_Pad1.15x1.40mm_HandSolder, symbol Device:R_Small_US
- removed R17, R18: 470, Resistor_SMD:R_0805_2012Metric_Pad1.15x1.40mm_HandSolder, symbol Device:R_Small_US
- removed R19: 470K, Resistor_SMD:R_0805_2012Metric_Pad1.15x1.40mm_HandSolder, symbol Device:R_Small_US
- removed R20, R22, R23, R24, R?: 22K, Resistor_SMD:R_0805_2012Metric_Pad1.15x1.40mm_HandSolder, symbol Device:R_Small_US
- removed R21: 2.2K, Resistor_SMD:R_0805_2012Metric_Pad1.15x1.40mm_HandSolder, symbol Device:R_Small_US
- removed R25, R?: 1ohm 1.2W, Resistor_THT:R_Axial_DIN0411_L9.9mm_D3.6mm_P15.24mm_Horizontal, symbol Device:R_Small_US
- removed R?: 220K, Resistor_SMD:R_0805_2012Metric_Pad1.15x1.40mm_HandSolder, symbol Device:R_Small_US
- removed TP4, TP5, TP8: TestPoint, TestPoint:TestPoint_Keystone_5000-5004_Miniature, symbol Connector:TestPoint
- removed U3, U?: LM1875, Package_TO_SOT_THT:TO-220-5_P3.4x3.7mm_StaggerOdd_Lead3.8mm_Vertical, symbol Amplifier_Audio:LM1875
- added C13, C14: 10uF, Capacitor_SMD:C_0805_2012Metric_Pad1.15x1.40mm_HandSolder, symbol Device:C_Small
- added U4: TPA3118AmplifierBoard, Arduino controlled radio:TPA3118_Board, symbol Arduino~Controlled~Radio:TPA3118AmplifierBoard
- C10, C11, C12: renamed from C?; footprint Capacitor_SMD:C_0805_2012Metric_Pad1.18x1.45mm_HandSolder -> Capacitor_SMD:C_0805_2012Metric_Pad1.15x1.40mm_HandSolder
- C15: value 10uF 16V -> 100uF; footprint Capacitor_SMD:CP_Elec_4x5.3 -> Capacitor_SMD:C_Elec_6.3x5.4
- C16: value 1uF -> .1 uF; footprint Capacitor_SMD:C_0805_2012Metric_Pad1.18x1.45mm_HandSolder -> Capacitor_SMD:C_0805_2012Metric_Pad1.15x1.40mm_HandSolder
- U3: renamed from U?; value LM358 -> TL082; footprint (none) -> Arduino controlled radio:TL082CDR
- U3: renamed from U?; value LM358 -> TL082
- gave numbers to parts that had none: 11
Connections:
- net labels removed: +5V
- wire segments 174 -> 76
Other:
- moved on the sheet: C10, C11, C12, J8, R11, R12, R13, R14, R15, R16, R17, R18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
